File: project/MUC.kicad_sch (KiCad schematic)
At the start: 33 parts, among them IC10 FAN5622SX, IC15 DRV2603RUNT, IC2 ESDALC6V1W5, IC6 AT25SL128A, IC9 NTS0104GU12, M1 NORA-B106, M2 Vibrator DC Motor, X1 DOCK, X10 M-, X3 GPIO0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

Commit message: - Add QR code library with link to the project - Change ISET resistor to 12k - Replace light sensor footprint with a version from our KiCad library - Rename the inner copper layers - Add KiBot file for production file generation - Import nPM1300 from test project - Remove pull down resistor from vibration driver IC enable - Split schematics into hierarical schematics - Add PCB variant for reduced sensor board - Add I2S microphone - Update all symbols and footprints
Signed-off-by: Daniel Kampert <DanielKampert@kampis-elektroecke.de>
Parts:
- removed TP1: RESET, TestPoint:TestPoint_Pad_D1.0mm, symbol Connector:TestPoint
- removed TP2: SCL, TestPoint:TestPoint_Pad_D1.0mm, symbol Connector:TestPoint
- removed TP3: SDA, TestPoint:TestPoint_Pad_D1.0mm, symbol Connector:TestPoint
- removed TP4: 3V3, TestPoint:TestPoint_Pad_D1.0mm, symbol Connector:TestPoint
- removed X3: GPIO0, TestPoint:TestPoint_Pad_1.0x1.0mm, symbol Connector_Generic:Conn_01x01
- removed X4: GPIO1, TestPoint:TestPoint_Pad_1.0x1.0mm, symbol Connector_Generic:Conn_01x01
- removed X5: GPIO2, TestPoint:TestPoint_Pad_1.0x1.0mm, symbol Connector_Generic:Conn_01x01
- removed X6: GPIO3, TestPoint:TestPoint_Pad_1.0x1.0mm, symbol Connector_Generic:Conn_01x01
- removed X7: GND, TestPoint:TestPoint_Pad_1.0x1.0mm, symbol Connector_Generic:Conn_01x01
- added BZ1: Buzzer, CUI Devices:CMT-322-65-SMT-TR, symbol Device:Buzzer
- added C12: 1u, Capacitor_SMD:C_0603_1608Metric, symbol Device:C_Small
- added C12: 200p, Capacitor_SMD:C_0603_1608Metric, symbol Device:C_Small
- added D1: BAS316, Diode_SMD:D_SOD-323, symbol Diode:BAS316
- added MK1: SPH0645LM4H-B, Knowles:SPH0645LM4H-6_3.5x2.65mm, symbol Knowles:SPH0645LM4H-B
- added Q1: BC817W, Package_TO_SOT_SMD:SOT-323_SC-70, symbol Transistor_BJT:BC817W
- added R12: 180R, Resistor_SMD:R_0603_1608Metric, symbol Device:R_Small
Connections:
- net GPIO3 is gone; now on net DRV_VIB_EN: M1.E9 (P1.05)
- net +1V8: now also C12.2, C12.2, MK1.5 (VDD)
- net BTN_2: now also M1.J7 (P1.10); no longer M1.H8 (P0.30)
- net BTN_3: now also M1.J8 (P0.28/AIN7); no longer M1.G8 (P1.12)
- net DRV_VIB_EN: no longer M1.F8 (P1.14)
- net GND: now also C12.1, C12.1, MK1.1 (WS), MK1.3 (GND), Q1.2 (E)
- net VBUS: no longer M1.B9 (VBUS)
- net BUZZER: now reaches M1.B6 (P0.01/XL2)
- net BUZZER: now also R12.1
- net BMI270-INT2: now reaches M1.G4 (P1.04)
- net BMI270-INT1: now reaches M1.G5 (P1.08)
- net PMIC-INT: now reaches M1.H9 (P1.11)
- net +BATT renamed VBAT
- net BMP581_INT renamed MIC_BCLK
- net MIC_BCLK: now also MK1.4 (BCLK)
- net DISPLAY_3V3 renamed VDD-Display
- net GPIO0: no longer names the net of M1.C8 (P0.22)
- net GPIO1: no longer names the net of M1.D8 (P0.04/AIN0)
- net GPIO2: no longer names the net of M1.E8 (P0.05/AIN1)
- net LIS-INT1 renamed MIC_SEL
- net MIC_SEL: now also MK1.2 (SEL)
- net LIS-INT2 renamed MIC_DATA
- net MIC_DATA: now also MK1.6 (DATA)
- new net: BZ1.2 (+), D1.2 (A), Q1.3 (C)
- new net: Q1.1 (B), R12.2
- new net +3V0: BZ1.1 (-), D1.1 (K)
- new net VBUS-MCU: M1.B9 (VBUS)
- no-connect marks 16 -> 19
Other:
- note added: "12k gives I_{LED} of <25 mA (max.)"
- note added: "1V8 <-> 3V3 level shifter"
- note added: "Buzzer"
- note added: "Can we use VUSB without USB lines?"
- note added: "Microphone"
- note removed: "1.8<->3.3 level shifter"
- note removed: "9.53k gives I_{LED} 30mA (max)"
- note removed: "GPIO"
- note removed: "Pull down all EN. Battery is connected directly to some of those ICs but since EN is pulled low and only set high by ANNA, they will be off when battery is low (NORA shut off)."
- note removed: "Test Points"
- moved on the sheet: C10, C12, C20, C5, C9, IC10, IC6, IC9, M2, R12, R6, R7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
