File: project/Power.kicad_sch (KiCad schematic)
At the start: 20 parts, among them IC101 nPM1300-QEXX, X101 BATTERY

Commit message: - Add RV-8263-C8 - Update CHANGELOG
Connections:
- net VBAT: now reaches C103.1, R103.1, X101.1 (Pin_1)
Changed lines of the file:
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@@
   (junction (at 193.04 95.25) (diameter 0) (color 0 0 0 0)
+  )
+  (junction (at 135.89 40.64) (diameter 0) (color 0 0 0 0)
   )
   (junction (at 201.93 59.69) (diameter 0) (color 0 0 0 0)
@@
     (stroke (width 0) (type default))
   )
+  (wire (pts (xy 135.89 39.37) (xy 135.89 40.64))
+    (stroke (width 0) (type default))
+  )
   (wire (pts (xy 165.1 77.47) (xy 168.91 77.47))
     (stroke (width 0) (type default))
@@
     (effects (font (size 1.27 1.27)) (justify left))
   )
+  (hierarchical_label "VBAT" (shape output) (at 135.89 39.37 90) (fields_autoplaced)
+    (effects (font (size 1.27 1.27)) (justify left))
+  )

Commit message: Fix different manufacturing issues
Parts:
- R103: Mfr. No. CR0603-J/-000ELF -> CR0402-J/-000GLF
Changed lines of the file:
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@@
       (effects (font (size 1.27 1.27)) hide)
     )
-    (property "Datasheet" "https://infocenter.nordicsemi.com/index.jsp?topic=%2Fstruct_pmic%2Fstruct%2Fnpm1300.html" (at 132.08 110.49 0)
+    (property "Datasheet" "https://docs.nordicsemi.com/category/npm1300-category" (at 132.08 110.49 0)
       (effects (font (size 1.27 1.27)) hide)
     )
@@
       (effects (font (size 1.27 1.27)) hide)
     )
-    (property "Mfr. No." "CR0603-J/-000ELF" (at 135.89 63.5 0)
-      (effects (font (size 1.27 1.27)) hide)
-    )
+    (property "Mfr. No." "CR0402-J/-000GLF" (at 135.89 63.5 0)
+      (effects (font (size 1.27 1.27)) hide)
+    )
