File: project/Power.kicad_sch (KiCad schematic)
At the start: 20 parts, among them IC101 nPM1300-QEXX, X101 BATTERY

Commit message: Rename Order. No. field in Order No.
Parts:
- C101, C110: Order No. (none) -> 581-0603YC105JAT2A; Order. No. 581-0603YC105JAT2A -> (none)
- C102: Order No. (none) -> 581-06035C104KAT2A; Order. No. 581-06035C104KAT2A -> (none)
- C103: Order No. (none) -> 581-06036D225KAT2A; Order. No. 581-06036D225KAT2A -> (none)
- C104, C105, C106, C107, C108, C109: Order No. (none) -> 346-CM105X5R106M25AT; Order. No. 346-CM105X5R106M25AT -> (none)
- IC101: Order No. (none) -> 949-NPM1300-QEAA-R7; Order. No. 949-NPM1300-QEAA-R7 -> (none)
- L101, L102: Order No. (none) -> 187-CIGT201610EH2R2MNE; Order. No. 187-CIGT201610EH2R2MNE -> (none)
- R101: Order No. (none) -> 603-RC0603FR-0747KL; Order. No. 603-RC0603FR-0747KL -> (none)
- R102: Order No. (none) -> 603-RC0603FR-07150KL; Order. No. 603-RC0603FR-07150KL -> (none)
- R103: Order No. (none) -> 652-CR0603-J/-000ELF; Order. No. 652-CR0603-J/-000ELF -> (none)
- X101: Order No. (none) -> 538-78171-0002; Order. No. 538-78171-0002 -> (none)
Changed lines of the file:
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@@
 			)
 		)
-		(property "Order. No." "581-0603YC105JAT2A"
+		(property "Order No." "581-0603YC105JAT2A"
 			(at 218.44 91.44 0)
 			(effects
@@
 			)
 		)
-		(property "Order. No." "187-CIGT201610EH2R2MNE"
-			(at 173.99 106.68 0)
-			(effects
-				(font
-					(size 1.27 1.27)
-				)
-				(hide yes)
-			)
-		)
-		(property "Order No." ""
+		(property "Order No." "187-CIGT201610EH2R2MNE"
 			(at 173.99 106.68 0)
 			(effects
@@
 			)
 		)
-		(property "Order. No." "581-0603YC105JAT2A"
+		(property "Order No." "581-0603YC105JAT2A"
 			(at 113.03 44.45 0)
 			(effects
@@
 			)
 		)
-		(property "Order. No." "346-CM105X5R106M25AT"
+		(property "Order No." "346-CM105X5R106M25AT"
 			(at 184.15 109.22 0)
 			(effects
@@
 			)
 		)
-		(property "Order. No." "603-RC0603FR-07150KL"
+		(property "Order No." "603-RC0603FR-07150KL"
 			(at 82.55 134.62 0)
 			(effects
@@
 			)
 		)
-		(property "Order. No." "346-CM105X5R106M25AT"
+		(property "Order No." "346-CM105X5R106M25AT"
 			(at 193.04 91.44 0)
 			(effects
@@
 			)
 		)
-		(property "Order. No." "603-RC0603FR-0747KL"
+		(property "Order No." "603-RC0603FR-0747KL"
 			(at 80.01 134.62 0)
 			(effects
@@
 			)
 		)
-		(property "Order. No." "949-NPM1300-QEAA-R7"
-			(at 132.08 107.95 0)
-			(effects
-				(font
-					(size 1.27 1.27)
-				)
-				(hide yes)
-			)
-		)
-		(property "Order No." ""
+		(property "Order No." "949-NPM1300-QEAA-R7"
 			(at 132.08 107.95 0)
 			(effects
@@
 			)
 		)
-		(property "Order. No." "346-CM105X5R106M25AT"
+		(property "Order No." "346-CM105X5R106M25AT"
 			(at 191.77 63.5 0)
 			(effects
@@
 			)
 		)
-		(property "Order. No." "187-CIGT201610EH2R2MNE"
-			(at 182.88 88.9 0)
-			(effects
-				(font
-					(size 1.27 1.27)
-				)
-				(hide yes)
-			)
-		)
-		(property "Order No." ""
+		(property "Order No." "187-CIGT201610EH2R2MNE"
 			(at 182.88 88.9 0)
 			(effects
@@
 			)
 		)
-		(property "Order. No." "538-78171-0002"
+		(property "Order No." "538-78171-0002"
 			(at 158.75 40.64 0)
 			(effects
@@
 			)
 		)
-		(property "Order. No." "652-CR0603-J/-000ELF"
+		(property "Order No." "652-CR0603-J/-000ELF"
 			(at 135.89 63.5 0)
 			(effects
@@
 			)
 		)
-		(property "Order. No." "346-CM105X5R106M25AT"
+		(property "Order No." "346-CM105X5R106M25AT"
 			(at 181.61 63.5 0)
 			(effects
@@
 			)
 		)
-		(property "Order. No." "581-06036D225KAT2A"
+		(property "Order No." "581-06036D225KAT2A"
 			(at 140.97 44.45 0)
 			(effects
@@
 			)
 		)
-		(property "Order. No." "346-CM105X5R106M25AT"
+		(property "Order No." "346-CM105X5R106M25AT"
 			(at 200.66 132.08 0)
 			(effects
@@
 			)
 		)
-		(property "Order. No." "581-06035C104KAT2A"
+		(property "Order No." "581-06035C104KAT2A"
 			(at 128.27 44.45 0)
 			(effects
@@
 			)
 		)
-		(property "Order. No." "346-CM105X5R106M25AT"
+		(property "Order No." "346-CM105X5R106M25AT"
 			(at 201.93 63.5 0)
 			(effects

Commit message: Display is now supplied with 3V0, add current consumption overview, vibration motor is now supplied with 3V0, add 0R series resistor for buzzer
Connections:
- net V_{DD}-Display: no longer names the net of C108.1, IC101.29 (LSOUT1/VOUTLDO1), TP103.1
Changed lines of the file:
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@@
-	(wire
-		(pts
-			(xy 200.66 127) (xy 203.2 127)
-		)
-		(stroke
-			(width 0)
-			(type default)
-		)
-	)
 	(wire
 		(pts
@@
 		(fields_autoplaced yes)
 		(effects
-			(font
-				(size 1.27 1.27)
-			)
-			(justify left)
-		)
-	)
-	(hierarchical_label "V_{DD}-Display"
-		(shape output)
-		(at 203.2 127 0)
-		(fields_autoplaced yes)
-		(effects
