File: project/Sensors.kicad_sch (KiCad schematic)
At the start: 21 parts, among them IC201 APDS-9306-065, IC202 BMI270, IC203 BMP581, IC204 LIS2MDLTR, IC205 BME688, Q201 DMG1013UW-7

Commit message: Change layer for PCB tables to User1
Parts:
- C201, C202, C203, C204, C206, C207, C210, C211, C212: Order Number 581-06035C104KAT2A -> (none); Order. No. (none) -> 581-06035C104KAT2A
- C208: Order Number 581-06033C224KAT2A -> (none); Order. No. (none) -> 581-06033C224KAT2A
- C209: Order Number 346-CM105X5R106M25AT -> (none); Order. No. (none) -> 346-CM105X5R106M25AT
- IC201: Order Number 630-APDS-9306-065 -> (none); Order. No. (none) -> 630-APDS-9306-065
- IC202: Order Number 262-BMI270 -> (none); Order. No. (none) -> 262-BMI270
- IC203: Order Number 262-BMP581 -> (none); Order. No. (none) -> 262-BMP581
- IC204: Order Number 511-LIS2MDLTR -> (none); Order. No. (none) -> 511-LIS2MDLTR
- IC205: Order Number 262-BME688 -> (none); Order. No. (none) -> 262-BME688
- MK201: Order Number 721-SPK0641HT4H-1 -> (none); Order. No. (none) -> 721-SPK0641HT4H-1
- Q201: Order Number 621-DMG1013UW-7 -> (none); Order. No. (none) -> 621-DMG1013UW-7
- R201: Order Number 603-RC0603FR-07150KL -> (none); Order. No. (none) -> 603-RC0603FR-07150KL
Changed lines of the file:
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@@
 			)
 		)
-		(property "Datasheet" "~"
+		(property "Datasheet" "https://www.mouser.de/datasheet/2/40/KGM_X7R-3223212.pdf"
 			(at 252.73 27.94 0)
 			(effects
@@
 			)
 		)
-		(property "Order Number" "581-06035C104KAT2A"
+		(property "CONFIG" ""
 			(at 252.73 27.94 0)
 			(effects
@@
 			)
 		)
-		(property "CONFIG" ""
+		(property "Order. No." "581-06035C104KAT2A"
 			(at 252.73 27.94 0)
 			(effects
@@
 			)
 		)
-		(property "Datasheet" "~"
+		(property "Datasheet" "https://www.mouser.de/datasheet/2/40/KGM_X7R-3223212.pdf"
 			(at 118.11 36.83 0)
 			(effects
@@
 			)
 		)
-		(property "Order Number" "581-06035C104KAT2A"
+		(property "CONFIG" ""
 			(at 118.11 36.83 0)
 			(effects
@@
 			)
 		)
-		(property "CONFIG" ""
+		(property "Order. No." "581-06035C104KAT2A"
 			(at 118.11 36.83 0)
 			(effects
@@
 			)
 		)
-		(property "Datasheet" "~"
+		(property "Datasheet" "https://www.mouser.de/datasheet/2/40/KGM_X7R-3223212.pdf"
 			(at 250.19 118.11 0)
 			(effects
@@
 			)
 		)
-		(property "Order Number" "581-06035C104KAT2A"
+		(property "CONFIG" ""
 			(at 250.19 118.11 0)
 			(effects
@@
 			)
 		)
-		(property "CONFIG" ""
+		(property "Order. No." "581-06035C104KAT2A"
 			(at 250.19 118.11 0)
 			(effects
@@
 			)
 		)
-		(property "Datasheet" "~"
+		(property "Datasheet" "https://www.mouser.de/datasheet/2/40/KGM_X7R-3223212.pdf"
 			(at 227.33 58.42 0)
 			(effects
@@
 			)
 		)
-		(property "Order Number" "581-06033C224KAT2A"
+		(property "CONFIG" ""
 			(at 227.33 58.42 0)
 			(effects
@@
 			)
 		)
-		(property "CONFIG" ""
+		(property "Order. No." "581-06033C224KAT2A"
 			(at 227.33 58.42 0)
 			(effects
@@
 			)
 		)
-		(property "Order Number" "262-BMI270"
+		(property "CONFIG" ""
 			(at 48.26 63.5 0)
 			(effects
@@
 			)
 		)
-		(property "CONFIG" ""
+		(property "Order. No." "262-BMI270"
 			(at 48.26 63.5 0)
 			(effects
@@
 			)
 		)
-		(property "Datasheet" "~"
+		(property "Datasheet" "https://www.mouser.de/datasheet/2/40/KGM_X7R-3223212.pdf"
 			(at 125.73 36.83 0)
 			(effects
@@
 			)
 		)
-		(property "Order Number" "581-06035C104KAT2A"
+		(property "CONFIG" ""
 			(at 125.73 36.83 0)
 			(effects
@@
 			)
 		)
-		(property "CONFIG" ""
+		(property "Order. No." "581-06035C104KAT2A"
 			(at 125.73 36.83 0)
 			(effects
@@
 			)
 		)
-		(property "Order Number" "621-DMG1013UW-7"
+		(property "CONFIG" "-ENV"
 			(at 80.01 146.05 0)
 			(effects
@@
 			)
 		)
-		(property "CONFIG" "-ENV"
+		(property "Order. No." "621-DMG1013UW-7"
 			(at 80.01 146.05 0)
 			(effects
@@
 			)
 		)
-		(property "Order Number" "630-APDS-9306-065"
+		(property "CONFIG" ""
 			(at 24.13 180.34 0)
 			(effects
@@
 			)
 		)
-		(property "CONFIG" ""
+		(property "Order. No." "630-APDS-9306-065"
 			(at 24.13 180.34 0)
 			(effects
@@
 			)
 		)
-		(property "Order Number" ""
-			(at 227.33 147.32 0)
-			(effects
-				(font
-					(size 1.27 1.27)
-				)
-				(hide yes)
-			)
-		)
 		(property "CONFIG" ""
 			(at 227.33 147.32 0)
@@
 			)
 		)
-		(property "Datasheet" "~"
+		(property "Datasheet" "https://www.mouser.de/datasheet/2/40/KGM_X7R-3223212.pdf"
 			(at 44.45 36.83 0)
 			(effects
@@
 			)
 		)
-		(property "Order Number" "581-06035C104KAT2A"
+		(property "CONFIG" ""
 			(at 44.45 36.83 0)
 			(effects
@@
 			)
 		)
-		(property "CONFIG" ""
+		(property "Order. No." "581-06035C104KAT2A"
 			(at 44.45 36.83 0)
 			(effects
@@
 			)
 		)
-		(property "Datasheet" "~"
+		(property "Datasheet" "https://www.mouser.de/datasheet/2/40/KGM_X7R-3223212.pdf"
 			(at 242.57 118.11 0)
 			(effects
@@
 			)
 		)
-		(property "Order Number" "581-06035C104KAT2A"
+		(property "CONFIG" ""
 			(at 242.57 118.11 0)
 			(effects
@@
 			)
 		)
-		(property "CONFIG" ""
+		(property "Order. No." "581-06035C104KAT2A"
 			(at 242.57 118.11 0)
 			(effects
@@
 			)
 		)
-		(property "Datasheet" "~"
+		(property "Datasheet" "https://www.mouser.de/datasheet/2/40/KGM_X7R-3223212.pdf"
 			(at 30.48 165.1 0)
 			(effects
@@
 			)
 		)
-		(property "Order Number" "581-06035C104KAT2A"
+		(property "CONFIG" ""
 			(at 30.48 165.1 0)
 			(effects
@@
 			)
 		)
-		(property "CONFIG" ""
+		(property "Order. No." "581-06035C104KAT2A"
 			(at 30.48 165.1 0)
 			(effects
@@
 			)
 		)
-		(property "Order Number" ""
-			(at 227.33 152.4 0)
-			(effects
-				(font
-					(size 1.27 1.27)
-				)
-				(hide yes)
-			)
-		)
 		(property "CONFIG" ""
 			(at 227.33 152.4 0)
@@
 			)
 		)
-		(property "Order Number" "511-LIS2MDLTR"
+		(property "CONFIG" ""
 			(at 248.92 50.8 0)
 			(effects
@@
 			)
 		)
-		(property "CONFIG" ""
+		(property "Order. No." "511-LIS2MDLTR"
 			(at 248.92 50.8 0)
 			(effects
@@
 			)
 		)
-		(property "Order Number" "603-RC0603FR-07150KL"
+		(property "CONFIG" "-ENV"
 			(at 71.12 142.24 0)
 			(effects
@@
 			)
 		)
-		(property "CONFIG" "-ENV"
+		(property "Order. No." "603-RC0603FR-07150KL"
 			(at 71.12 142.24 0)
 			(effects
@@
 			)
 		)
-		(property "Order Number" "262-BME688"
+		(property "CONFIG" ""
 			(at 246.38 142.24 0)
 			(effects
@@
 			)
 		)
-		(property "CONFIG" ""
+		(property "Order. No." "262-BME688"
 			(at 246.38 142.24 0)
 			(effects
@@
 			)
 		)
-		(property "Order Number" "721-SPK0641HT4H-1"
+		(property "CONFIG" "-ENV"
 			(at 80.01 177.8 0)
 			(effects
@@
 			)
 		)
-		(property "CONFIG" "-ENV"
+		(property "Order. No." "721-SPK0641HT4H-1"
 			(at 80.01 177.8 0)
 			(effects
@@
 			)
 		)
-		(property "Datasheet" "~"
+		(property "Datasheet" "https://www.mouser.de/datasheet/2/40/KGM_X7R-3223212.pdf"
 			(at 83.82 160.02 0)
 			(effects
@@
 			)
 		)
-		(property "Order Number" "581-06035C104KAT2A"
+		(property "CONFIG" ""
 			(at 83.82 160.02 0)
 			(effects
@@
 			)
 		)
-		(property "CONFIG" ""
+		(property "Order. No." "581-06035C104KAT2A"
 			(at 83.82 160.02 0)
 			(effects
@@
 			)
 		)
-		(property "Order Number" "262-BMP581"
+		(property "CONFIG" ""
 			(at 121.92 63.5 0)
 			(effects
@@
 			)
 		)
-		(property "CONFIG" ""
+		(property "Order. No." "262-BMP581"
 			(at 121.92 63.5 0)
 			(effects
@@
 			)
 		)
-		(property "Datasheet" "~"
+		(property "Datasheet" "https://www.mouser.de/datasheet/2/40/KGM_X7R-3223212.pdf"
 			(at 52.07 36.83 0)
 			(effects
@@
 			)
 		)
-		(property "Order Number" "581-06035C104KAT2A"
+		(property "CONFIG" ""
 			(at 52.07 36.83 0)
 			(effects
@@
 			)
 		)
-		(property "CONFIG" ""
+		(property "Order. No." "581-06035C104KAT2A"
 			(at 52.07 36.83 0)
 			(effects
@@
 			)
 		)
-		(property "Datasheet" "~"
+		(property "Datasheet" "https://www.mouser.de/datasheet/2/40/CM_Series_e-2835982.pdf"
 			(at 245.11 27.94 0)
 			(effects
@@
 			)
 		)
-		(property "Order Number" "346-CM105X5R106M25AT"
+		(property "CONFIG" ""
 			(at 245.11 27.94 0)
 			(effects
@@
 			)
 		)
-		(property "CONFIG" ""
+		(property "Order. No." "346-CM105X5R106M25AT"
 			(at 245.11 27.94 0)
 			(effects

Commit message: - Switch to a local KiCad library
Parts:
- IC202: footprint Package_LGA_Kampi:Bosch_LGA-14_3x2.5mm_P0.5mm_LayoutBorder3x4y -> Package_LGA:Bosch_LGA-14_3x2.5mm_P0.5mm_LayoutBorder3x4y; symbol Bosch_Kampi:BMI270 -> Bosch:BMI270
- IC203: footprint Package_LGA_Kampi:Bosch_LGA-10_2x2mm_P0.5mm_ClockwisePinNumbering -> Package_LGA:Bosch_LGA-10_2x2mm_P0.5mm_ClockwisePinNumbering; symbol Bosch_Kampi:BMP581 -> Bosch:BMP581
- IC204: footprint Package_LGA_Kampi:LGA-12_2x2mm_P0.5mm -> Package_LGA:LGA-12_2x2mm_P0.5mm
- IC205: footprint Package_LGA_Kampi:Bosch_LGA-8_3x3mm_P0.8mm_ClockwisePinNumbering -> Package_LGA:Bosch_LGA-8_3x3mm_P0.8mm_ClockwisePinNumbering; symbol Bosch_Kampi:BME688 -> Bosch:BME688
Changed lines of the file:
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@@
 	)
 	(symbol
-		(lib_id "Bosch_Kampi:BMI270")
+		(lib_id "Bosch:BMI270")
 		(at 48.26 63.5 0)
 		(unit 1)
@@
 			)
 		)
-		(property "Footprint" "Package_LGA_Kampi:Bosch_LGA-14_3x2.5mm_P0.5mm_LayoutBorder3x4y"
+		(property "Footprint" "Package_LGA:Bosch_LGA-14_3x2.5mm_P0.5mm_LayoutBorder3x4y"
 			(at 48.26 63.5 0)
 			(effects
@@
 		)
 		(property "Order. No." "262-BMI270"
+			(at 48.26 63.5 0)
+			(effects
+				(font
+					(size 1.27 1.27)
+				)
+				(hide yes)
+			)
+		)
+		(property "Order No." ""
 			(at 48.26 63.5 0)
 			(effects
@@
 			)
 		)
-		(property "Footprint" "Package_LGA_Kampi:LGA-12_2x2mm_P0.5mm"
+		(property "Footprint" "Package_LGA:LGA-12_2x2mm_P0.5mm"
 			(at 248.92 50.8 0)
 			(effects
@@
 		)
 		(property "Order. No." "511-LIS2MDLTR"
+			(at 248.92 50.8 0)
+			(effects
+				(font
+					(size 1.27 1.27)
+				)
+				(hide yes)
+			)
+		)
+		(property "Order No." ""
 			(at 248.92 50.8 0)
 			(effects
@@
 	)
 	(symbol
-		(lib_id "Bosch_Kampi:BME688")
+		(lib_id "Bosch:BME688")
 		(at 246.38 142.24 0)
 		(unit 1)
@@
 			)
 		)
-		(property "Footprint" "Package_LGA_Kampi:Bosch_LGA-8_3x3mm_P0.8mm_ClockwisePinNumbering"
-			(at 283.21 153.67 0)
+		(property "Footprint" "Package_LGA:Bosch_LGA-8_3x3mm_P0.8mm_ClockwisePinNumbering"
+			(at 246.38 142.24 0)
 			(effects
 				(font
@@
 		)
 		(property "Datasheet" "https://www.bosch-sensortec.com/media/boschsensortec/downloads/datasheets/bst-bme688-ds000.pdf"
-			(at 246.38 147.32 0)
-			(effects
-				(font
-					(size 1.27 1.27)
-				)
-				(hide yes)
-			)
-		)
-		(property "Description" ""
+			(at 246.38 142.24 0)
+			(effects
+				(font
+					(size 1.27 1.27)
+				)
+				(hide yes)
+			)
+		)
+		(property "Description" "4-in-1 sensor, gas, humidity, pressure, temperature, I2C and SPI interface, 1.71-3.6V, LGA-8"
 			(at 246.38 142.24 0)
 			(effects
@@
 		)
 		(property "Order. No." "262-BME688"
+			(at 246.38 142.24 0)
+			(effects
+				(font
+					(size 1.27 1.27)
+				)
+				(hide yes)
+			)
+		)
+		(property "Order No." ""
 			(at 246.38 142.24 0)
 			(effects
@@
 	)
 	(symbol
-		(lib_id "Bosch_Kampi:BMP581")
+		(lib_id "Bosch:BMP581")
 		(at 121.92 63.5 0)
 		(unit 1)
@@
 			)
 		)
-		(property "Footprint" "Package_LGA_Kampi:Bosch_LGA-10_2x2mm_P0.5mm_ClockwisePinNumbering"
-			(at 121.92 62.23 0)
+		(property "Footprint" "Package_LGA:Bosch_LGA-10_2x2mm_P0.5mm_ClockwisePinNumbering"
+			(at 121.92 63.5 0)
 			(effects
 				(font
@@
 		)
 		(property "Datasheet" "https://www.bosch-sensortec.com/media/boschsensortec/downloads/datasheets/bst-bmp581-ds004.pdf"
-			(at 121.92 62.23 0)
+			(at 121.92 63.5 0)
 			(effects
 				(font
@@
 			(at 121.92 63.5 0)
 			(effects
+				(font
+					(size 1.27 1.27)
+				)
+				(hide yes)
+			)
+		)
+		(property "Order No." ""
+			(at 121.92 63.5 0)
+			(effects

Commit message: Rename Order. No. field in Order No.
Parts:
- C201, C202, C203, C204, C206, C207, C210, C211, C212: Order No. (none) -> 581-06035C104KAT2A; Order. No. 581-06035C104KAT2A -> (none)
- C208: Order No. (none) -> 581-06033C224KAT2A; Order. No. 581-06033C224KAT2A -> (none)
- C209: Order No. (none) -> 346-CM105X5R106M25AT; Order. No. 346-CM105X5R106M25AT -> (none)
- IC201: Order No. (none) -> 630-APDS-9306-065; Order. No. 630-APDS-9306-065 -> (none)
- IC202: Order No. (none) -> 262-BMI270; Order. No. 262-BMI270 -> (none)
- IC203: Order No. (none) -> 262-BMP581; Order. No. 262-BMP581 -> (none)
- IC204: Order No. (none) -> 511-LIS2MDLTR; Order. No. 511-LIS2MDLTR -> (none)
- IC205: Order No. (none) -> 262-BME688; Order. No. 262-BME688 -> (none)
- MK201: Order No. (none) -> 721-SPK0641HT4H-1; Order. No. 721-SPK0641HT4H-1 -> (none)
- Q201: Order No. (none) -> 621-DMG1013UW-7; Order. No. 621-DMG1013UW-7 -> (none)
- R201: Order No. (none) -> 603-RC0603FR-07150KL; Order. No. 603-RC0603FR-07150KL -> (none)
Changed lines of the file:
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@@
 			)
 		)
-		(property "Order. No." "581-06035C104KAT2A"
+		(property "Order No." "581-06035C104KAT2A"
 			(at 252.73 27.94 0)
 			(effects
@@
 			)
 		)
-		(property "Order. No." "581-06035C104KAT2A"
+		(property "Order No." "581-06035C104KAT2A"
 			(at 118.11 36.83 0)
 			(effects
@@
 			)
 		)
-		(property "Order. No." "581-06035C104KAT2A"
+		(property "Order No." "581-06035C104KAT2A"
 			(at 250.19 118.11 0)
 			(effects
@@
 			)
 		)
-		(property "Order. No." "581-06033C224KAT2A"
+		(property "Order No." "581-06033C224KAT2A"
 			(at 227.33 58.42 0)
 			(effects
@@
 			)
 		)
-		(property "Order. No." "262-BMI270"
-			(at 48.26 63.5 0)
-			(effects
-				(font
-					(size 1.27 1.27)
-				)
-				(hide yes)
-			)
-		)
-		(property "Order No." ""
+		(property "Order No." "262-BMI270"
 			(at 48.26 63.5 0)
 			(effects
@@
 			)
 		)
-		(property "Order. No." "581-06035C104KAT2A"
+		(property "Order No." "581-06035C104KAT2A"
 			(at 125.73 36.83 0)
 			(effects
@@
 			)
 		)
-		(property "Order. No." "621-DMG1013UW-7"
+		(property "Order No." "621-DMG1013UW-7"
 			(at 80.01 146.05 0)
 			(effects
@@
 			)
 		)
-		(property "Order. No." "630-APDS-9306-065"
+		(property "Order No." "630-APDS-9306-065"
 			(at 24.13 180.34 0)
 			(effects
@@
 			)
 		)
-		(property "Order. No." "581-06035C104KAT2A"
+		(property "Order No." "581-06035C104KAT2A"
 			(at 44.45 36.83 0)
 			(effects
@@
 			)
 		)
-		(property "Order. No." "581-06035C104KAT2A"
+		(property "Order No." "581-06035C104KAT2A"
 			(at 242.57 118.11 0)
 			(effects
@@
 			)
 		)
-		(property "Order. No." "581-06035C104KAT2A"
+		(property "Order No." "581-06035C104KAT2A"
 			(at 30.48 165.1 0)
 			(effects
@@
 			)
 		)
-		(property "Order. No." "511-LIS2MDLTR"
-			(at 248.92 50.8 0)
-			(effects
-				(font
-					(size 1.27 1.27)
-				)
-				(hide yes)
-			)
-		)
-		(property "Order No." ""
+		(property "Order No." "511-LIS2MDLTR"
 			(at 248.92 50.8 0)
 			(effects
@@
 			)
 		)
-		(property "Order. No." "603-RC0603FR-07150KL"
+		(property "Order No." "603-RC0603FR-07150KL"
 			(at 71.12 142.24 0)
 			(effects
@@
 			)
 		)
-		(property "Order. No." "262-BME688"
-			(at 246.38 142.24 0)
-			(effects
-				(font
-					(size 1.27 1.27)
-				)
-				(hide yes)
-			)
-		)
-		(property "Order No." ""
+		(property "Order No." "262-BME688"
 			(at 246.38 142.24 0)
 			(effects
@@
 			)
 		)
-		(property "Order. No." "721-SPK0641HT4H-1"
+		(property "Order No." "721-SPK0641HT4H-1"
 			(at 80.01 177.8 0)
 			(effects
@@
 			)
 		)
-		(property "Order. No." "581-06035C104KAT2A"
+		(property "Order No." "581-06035C104KAT2A"
 			(at 83.82 160.02 0)
 			(effects
@@
 			)
 		)
-		(property "Order. No." "262-BMP581"
-			(at 121.92 63.5 0)
-			(effects
-				(font
-					(size 1.27 1.27)
-				)
-				(hide yes)
-			)
-		)
-		(property "Order No." ""
+		(property "Order No." "262-BMP581"
 			(at 121.92 63.5 0)
 			(effects
@@
 			)
 		)
-		(property "Order. No." "581-06035C104KAT2A"
+		(property "Order No." "581-06035C104KAT2A"
 			(at 52.07 36.83 0)
 			(effects
@@
 			)
 		)
-		(property "Order. No." "346-CM105X5R106M25AT"
+		(property "Order No." "346-CM105X5R106M25AT"
 			(at 245.11 27.94 0)
 			(effects

Commit message: Fix wrong footprint path in symbols, add new vibration motor to PCB
Changed lines of the file:
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@@
 	)
 	(junction
-		(at 246.38 156.21)
-		(diameter 0)
-		(color 0 0 0 0)
-	)
-	(junction
 		(at 247.65 114.3)
 		(diameter 0)
@@
 	)
 	(junction
-		(at 48.26 81.28)
-		(diameter 0)
-		(color 0 0 0 0)
-	)
-	(junction
 		(at 80.01 156.21)
 		(diameter 0)
@@
 	)
 	(junction
-		(at 248.92 62.23)
-		(diameter 0)
-		(color 0 0 0 0)
-	)
-	(junction
 		(at 247.65 24.13)
 		(diameter 0)
@@
 	)
 	(junction
-		(at 121.92 81.28)
-		(diameter 0)
-		(color 0 0 0 0)
-	)
-	(junction
 		(at 245.11 114.3)
 		(diameter 0)
@@
 	)
 	(junction
-		(at 80.01 187.96)
-		(diameter 0)
-		(color 0 0 0 0)
-	)
-	(junction
 		(at 227.33 148.59)
 		(diameter 0)
@@
 	(wire
 		(pts
-			(xy 78.74 187.96) (xy 80.01 187.96)
-		)
-		(stroke
-			(width 0)
-			(type default)
-		)
-	)
-	(wire
-		(pts
 			(xy 245.11 114.3) (xy 245.11 129.54)
 		)
@@
 	(wire
 		(pts
-			(xy 119.38 80.01) (xy 119.38 81.28)
-		)
-		(stroke
-			(width 0)
-			(type default)
-		)
-	)
-	(wire
-		(pts
-			(xy 46.99 81.28) (xy 48.26 81.28)
-		)
-		(stroke
-			(width 0)
-			(type default)
-		)
-	)
-	(wire
-		(pts
-			(xy 81.28 187.96) (xy 81.28 186.69)
-		)
-		(stroke
-			(width 0)
-			(type default)
-		)
-	)
-	(wire
-		(pts
 			(xy 60.96 63.5) (xy 66.04 63.5)
 		)
@@
 	(wire
 		(pts
-			(xy 121.92 81.28) (xy 121.92 82.55)
-		)
-		(stroke
-			(width 0)
-			(type default)
-		)
-	)
-	(wire
-		(pts
 			(xy 125.73 33.02) (xy 123.19 33.02)
 		)
@@
 	(wire
 		(pts
-			(xy 83.82 162.56) (xy 83.82 163.83)
+			(xy 80.01 186.69) (xy 80.01 189.23)
 		)
 		(stroke
@@
 	(wire
 		(pts
-			(xy 49.53 80.01) (xy 49.53 81.28)
+			(xy 83.82 162.56) (xy 83.82 163.83)
 		)
 		(stroke
@@
 	(wire
 		(pts
-			(xy 248.92 63.5) (xy 248.92 62.23)
+			(xy 248.92 60.96) (xy 248.92 63.5)
 		)
 		(stroke
@@
 	(wire
 		(pts
-			(xy 247.65 156.21) (xy 246.38 156.21)
-		)
-		(stroke
-			(width 0)
-			(type default)
-		)
-	)
-	(wire
-		(pts
 			(xy 125.73 39.37) (xy 125.73 40.64)
 		)
@@
 	(wire
 		(pts
-			(xy 80.01 187.96) (xy 81.28 187.96)
-		)
-		(stroke
-			(width 0)
-			(type default)
-		)
-	)
-	(wire
-		(pts
 			(xy 62.23 67.31) (xy 60.96 67.31)
 		)
@@
 	(wire
 		(pts
-			(xy 78.74 186.69) (xy 78.74 187.96)
-		)
-		(stroke
-			(width 0)
-			(type default)
-		)
-	)
-	(wire
-		(pts
 			(xy 91.44 173.99) (xy 92.71 173.99)
 		)
@@
 	(wire
 		(pts
-			(xy 48.26 81.28) (xy 48.26 82.55)
+			(xy 48.26 80.01) (xy 48.26 82.55)
 		)
 		(stroke
@@
 		)
 	)
-	(wire
-		(pts
-			(xy 246.38 156.21) (xy 246.38 157.48)
-		)
-		(stroke
-			(width 0)
-			(type default)
-		)
-	)
 	(polyline
 		(pts
@@
 	(wire
 		(pts
-			(xy 247.65 60.96) (xy 247.65 62.23)
-		)
-		(stroke
-			(width 0)
-			(type default)
-		)
-	)
-	(wire
-		(pts
 			(xy 46.99 33.02) (xy 44.45 33.02)
 		)
@@
 	(wire
 		(pts
-			(xy 46.99 80.01) (xy 46.99 81.28)
-		)
-		(stroke
-			(width 0)
-			(type default)
-		)
-	)
-	(wire
-		(pts
 			(xy 246.38 114.3) (xy 245.11 114.3)
 		)
@@
 	(wire
 		(pts
-			(xy 248.92 62.23) (xy 247.65 62.23)
-		)
-		(stroke
-			(width 0)
-			(type default)
-		)
-	)
-	(wire
-		(pts
 			(xy 232.41 144.78) (xy 233.68 144.78)
 		)
@@
 	(wire
 		(pts
-			(xy 245.11 156.21) (xy 246.38 156.21)
-		)
-		(stroke
-			(width 0)
-			(type default)
-		)
-	)
-	(wire
-		(pts
 			(xy 250.19 24.13) (xy 250.19 38.1)
 		)
@@
 	(wire
 		(pts
-			(xy 124.46 81.28) (xy 121.92 81.28)
-		)
-		(stroke
-			(width 0)
-			(type default)
-		)
-	)
-	(wire
-		(pts
 			(xy 66.04 63.5) (xy 66.04 59.69)
 		)
@@
 	(wire
 		(pts
-			(xy 245.11 154.94) (xy 245.11 156.21)
-		)
-		(stroke
-			(width 0)
-			(type default)
-		)
-	)
-	(wire
-		(pts
 			(xy 52.07 33.02) (xy 52.07 34.29)
 		)
@@
 	(wire
 		(pts
-			(xy 80.01 187.96) (xy 80.01 189.23)
-		)
-		(stroke
-			(width 0)
-			(type default)
-		)
-	)
-	(wire
-		(pts
 			(xy 34.29 180.34) (xy 35.56 180.34)
 		)
@@
 	(wire
 		(pts
-			(xy 49.53 81.28) (xy 48.26 81.28)
-		)
-		(stroke
-			(width 0)
-			(type default)
-		)
-	)
-	(wire
-		(pts
-			(xy 247.65 154.94) (xy 247.65 156.21)
-		)
-		(stroke
-			(width 0)
-			(type default)
-		)
-	)
-	(wire
-		(pts
-			(xy 121.92 80.01) (xy 121.92 81.28)
+			(xy 121.92 80.01) (xy 121.92 82.55)
 		)
 		(stroke
@@
 	(wire
 		(pts
-			(xy 121.92 81.28) (xy 119.38 81.28)
+			(xy 208.28 49.53) (xy 208.28 50.8)
 		)
 		(stroke
@@
 	(wire
 		(pts
-			(xy 208.28 49.53) (xy 208.28 50.8)
+			(xy 34.29 60.96) (xy 35.56 60.96)
 		)
 		(stroke
@@
 	(wire
 		(pts
-			(xy 34.29 60.96) (xy 35.56 60.96)
+			(xy 125.73 33.02) (xy 125.73 34.29)
 		)
 		(stroke
@@
 	(wire
 		(pts
-			(xy 125.73 33.02) (xy 125.73 34.29)
+			(xy 246.38 154.94) (xy 246.38 157.48)
 		)
 		(stroke
@@
 	(wire
 		(pts
-			(xy 248.92 62.23) (xy 250.19 62.23)
-		)
-		(stroke
-			(width 0)
-			(type default)
-		)
-	)
-	(wire
-		(pts
 			(xy 245.11 25.4) (xy 245.11 24.13)
 		)
@@
 	(wire
 		(pts
-			(xy 124.46 80.01) (xy 124.46 81.28)
-		)
-		(stroke
-			(width 0)
-			(type default)
-		)
-	)
-	(wire
-		(pts
 			(xy 71.12 138.43) (xy 71.12 139.7)
 		)
@@
 		)
 	)
-	(wire
-		(pts
-			(xy 250.19 62.23) (xy 250.19 60.96)
-		)
-		(stroke
-			(width 0)
-			(type default)
-		)
-	)
 	(text "Gas, Pressure, Temperature\n& Humidity"
 		(exclude_from_sim no)
@@
 			)
 		)
-		(property "Datasheet" "https://www.knowles.com/docs/default-source/model-downloads/spk0641ht4h-1-rev-a.pdf"
+		(property "Datasheet" "https://www.knowles.com/docs/default-source/default-document-library/sph0645lm4h-1-datasheet.pdf"
 			(at 80.01 177.8 0)
 			(effects
@@
 			)
 		)
-		(property "Description" ""
+		(property "Description" "Digital MEMS Microphone"
 			(at 80.01 177.8 0)
 			(effects

Commit message: Fix different documentation issues
Parts:
- Q201: Mfr. ROHM Semiconductor -> Diodes Incorporated
Changed lines of the file:
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@@
 			)
 		)
-		(property "Mfr." "ROHM Semiconductor"
+		(property "Mfr." "Diodes Incorporated"
 			(at 80.01 146.05 0)
 			(effects
